Commit message: updates with yolo service

File: description/xacro/camera.xacro (robot description, xacro)
@@ -11,5 +11,5 @@
                 <box size="0.010 0.03 0.03"/>
             </geometry>
-            <material name="black"/>
+            <material name="Black"/>
         </visual>
         <visual>
@@ -18,5 +18,5 @@
                 <cylinder radius="0.002" length="0.1"/>
             </geometry>
-            <material name="black"/>
+            <material name="Black"/>
         </visual>
     </link>

File: description/xacro/lidar.xacro (robot description, xacro)
@@ -18,5 +18,5 @@
                 <cylinder radius="0.01" length="0.1"/>
             </geometry>
-            <material name="black"/>
+            <material name="Black"/>
         </visual>
         <collision>
