Commit message: add 2 RGB cameras

File: description/xacro/right_camera.xacro (robot description, xacro)
@@ -1,10 +1,10 @@
 <?xml version="1.0"?>
 <robot xmlns:xacro="http://www.ros.org/wiki/xacro" >
-    <joint name="camera_joint" type="fixed">
+    <joint name="right_camera_joint" type="fixed">
         <parent link="chassis"/>
-        <child link="camera_link"/>
-        <origin xyz="0.276 0 0.181" rpy="0 0 0"/>
+        <child link="right_camera_link"/>
+        <origin xyz="0.276 0.1 0.181" rpy="0 0 0"/>
     </joint>
-    <link name="camera_link">
+    <link name="right_camera_link">
         <visual>
             <geometry>
@@ -21,13 +21,13 @@
         </visual>
     </link>
-    <joint name="camera_optical_joint" type="fixed">
-        <parent link="camera_link"/>
-        <child link="camera_link_optical"/>
+    <joint name="right_camera_optical_joint" type="fixed">
+        <parent link="right_camera_link"/>
+        <child link="right_camera_link_optical"/>
         <origin xyz="0 0 0" rpy="${-pi/2} 0 ${-pi/2}"/>
     </joint>
-    <link name="camera_link_optical"></link>
-    <gazebo reference="camera_link">
+    <link name="right_camera_link_optical"></link>
+    <gazebo reference="right_camera_link">
         <material>Gazebo/Black</material>
-        <sensor name="camera" type="camera">
+        <sensor name="right_camera" type="camera">
             <pose> 0 0 0 0 0 0 </pose>
             <visualize>true</visualize>
@@ -45,6 +45,7 @@
                 </clip>
             </camera>
-            <plugin name="camera_controller" filename="libgazebo_ros_camera.so">
-                <frame_name>camera_link_optical</frame_name>
+            <plugin name="right_camera_controller" filename="libgazebo_ros_camera.so">
+                <robotNamespace>right_camera</robotNamespace>
+                <frame_name>right_camera_link_optical</frame_name>
             </plugin>
         </sensor>

File: description/xacro/robot_core.xacro (robot description, xacro)
@@ -4,5 +4,6 @@
     <xacro:include filename="$(find mobile_robot)/description/xacro/inertial_macros.xacro" />
     <xacro:include filename="$(find mobile_robot)/description/xacro/lidar.xacro" />
-    <xacro:include filename="$(find mobile_robot)/description/xacro/camera.xacro" />
+    <xacro:include filename="$(find mobile_robot)/description/xacro/right_camera.xacro" />
+    <xacro:include filename="$(find mobile_robot)/description/xacro/left_camera.xacro" />
     <!-- Base link -->
     <link name="base_link"></link>
