Commit message: add 4 wheels that can be controled individualy

File: description/xacro/colors.xacro (robot description, xacro)
@@ -1,14 +1,14 @@
 <?xml version="1.0"?>
 <robot xmlns:xacro="http://www.ros.org/wiki/xacro"  name="robot">
-    <material name="White">
+    <material name="white">
         <color rgba="1 1 1 1"/>
     </material>
-    <material name="Red">
+    <material name="red">
         <color rgba="1 0 0 1"/>
     </material>
-    <material name="Blue">
+    <material name="blue">
         <color rgba="0 0 1 1"/>
     </material>
-    <material name="Black">
+    <material name="black">
         <color rgba="0 0 0 1"/>
     </material>

File: description/xacro/gazebo_control.xacro (robot description, xacro)
@@ -2,8 +2,12 @@
 <robot xmlns:xacro="http://www.ros.org/wiki/xacro">
     <gazebo>
-        <plugin name="motor_contro" filename="libgazebo_ros_diff_drive.so">
-            <!-- Wheels -->
-            <left_joint>left_wheel_joint</left_joint>
-            <right_joint>right_wheel_joint</right_joint>
+        <plugin name="motor_control" filename="libgazebo_ros_diff_drive.so">
+            <!-- Front Wheels -->
+            <left_joint>front_left_wheel_joint</left_joint>
+            <right_joint>front_right_wheel_joint</right_joint>
+            <!-- Rear Wheels -->
+            <left_rear_joint>rear_left_wheel_joint</left_rear_joint>
+            <right_rear_joint>rear_right_wheel_joint</right_rear_joint>
+            <!-- Wheel Configuration -->
             <wheel_separation>0.35</wheel_separation>
             <wheel_diameter>0.1</wheel_diameter>
@@ -14,7 +18,11 @@
             <odometry_frame>odom</odometry_frame>
             <robot_base_frame>base_link</robot_base_frame>
+            <!-- Publishing Options -->
             <publish_odom>true</publish_odom>
             <publish_odom_tf>true</publish_odom_tf>
             <publish_wheel_tf>true</publish_wheel_tf>
+            <!-- Additional Parameters for 4 Wheels -->
+            <legacyMode>false</legacyMode>
+            <updateRate>50.0</updateRate>
         </plugin>
     </gazebo>

File: description/xacro/left_camera.xacro (robot description, xacro)
@@ -11,5 +11,5 @@
                 <box size="0.010 0.03 0.03"/>
             </geometry>
-            <material name="Black"/>
+            <material name="black"/>
         </visual>
         <visual>
@@ -18,5 +18,5 @@
                 <cylinder radius="0.002" length="0.1"/>
             </geometry>
-            <material name="Black"/>
+            <material name="black"/>
         </visual>
     </link>

File: description/xacro/lidar.xacro (robot description, xacro)
@@ -11,5 +11,5 @@
                 <cylinder radius="0.05" length="0.04"/>
             </geometry>
-            <material name="Red"/>
+            <material name="red"/>
         </visual>
         <visual>
@@ -18,5 +18,5 @@
                 <cylinder radius="0.01" length="0.1"/>
             </geometry>
-            <material name="Black"/>
+            <material name="black"/>
         </visual>
         <collision>

File: description/xacro/right_camera.xacro (robot description, xacro)
@@ -11,5 +11,5 @@
                 <box size="0.010 0.03 0.03"/>
             </geometry>
-            <material name="Black"/>
+            <material name="black"/>
         </visual>
         <visual>
@@ -18,5 +18,5 @@
                 <cylinder radius="0.002" length="0.1"/>
             </geometry>
-            <material name="Black"/>
+            <material name="black"/>
         </visual>
     </link>

File: description/xacro/robot_core.xacro (robot description, xacro)
@@ -6,4 +6,6 @@
     <xacro:include filename="$(find mobile_robot)/description/xacro/right_camera.xacro" />
     <xacro:include filename="$(find mobile_robot)/description/xacro/left_camera.xacro" />
+    <xacro:include filename="$(find mobile_robot)/description/xacro/left_wheels.xacro" />
+    <xacro:include filename="$(find mobile_robot)/description/xacro/right_wheels.xacro" />
     <!-- Base link -->
     <link name="base_link"></link>
@@ -20,5 +22,5 @@
                 <box size="0.3 0.3 0.15" />
             </geometry>
-            <material name="White" />
+            <material name="white" />
         </visual>
         <collision>
@@ -35,83 +37,3 @@
         <material>Gazebo/White</material>
     </gazebo>
-    <!-- Wheels -->
-    <!-- Left wheel -->
-    <joint name="left_wheel_joint" type="continuous">
-        <parent link="base_link" />
-        <child link="left_wheel" />
-        <origin xyz="0 0.175 0"  rpy="-${pi/2} 0 0"/>
-        <axis xyz= "0 0 1" />
-    </joint>
-    <link name="left_wheel">
-        <visual>
-            <geometry>
-                <cylinder radius="0.05" length="0.04" />
-            </geometry>
-            <material name="Black" />
-        </visual>
-        <collision>
-            <geometry>
-                <cylinder radius="0.05" length="0.04" />
-            </geometry>
-        </collision>
-        <xacro:inertial_cylinder mass="0.1" length="0.04" radius="0.05">
-            <origin xyz="0 0 0" rpy="0 0 0"/>
-        </xacro:inertial_cylinder>
-    </link>
-    <gazebo reference="left_wheel">
-        <material>Gazebo/Black</material>
-    </gazebo>
-    <!-- Right wheel -->
-    <joint name="right_wheel_joint" type="continuous">
-        <parent link="base_link" />
-        <child link="right_wheel" />
-        <origin xyz="0 -0.175 0"  rpy="${pi/2} 0 0"/>
-        <axis xyz= "0 0 -1" />
-    </joint>
-    <link name="right_wheel">
-        <visual>
-            <geometry>
-                <cylinder radius="0.05" length="0.04" />
-            </geometry>
-            <material name="Black" />
-        </visual>
-        <collision>
-            <geometry>
-                <cylinder radius="0.05" length="0.04" />
-            </geometry>
-        </collision>
-        <xacro:inertial_cylinder mass="0.1" length="0.04" radius="0.05">
-            <origin xyz="0 0 0" rpy="0 0 0"/>
-        </xacro:inertial_cylinder>
-    </link>
-    <gazebo reference="right_wheel">
-        <material>Gazebo/Black</material>
-    </gazebo>
-    <!-- Caster wheel -->
-    <joint name="caster_wheel_joint" type="fixed">
-        <parent link="chassis" />
-        <child link="caster_wheel" />
-        <origin xyz="0.24 0 0"/>
-    </joint>
-    <link name="caster_wheel">
-        <visual>
-            <geometry>
-                <sphere radius="0.05"/>
-            </geometry>
-            <material name="Black" />
-        </visual>
-        <collision>
-            <geometry>
-                <sphere radius="0.05"/>
-            </geometry>
-        </collision>
-        <xacro:inertial_sphere mass="0.1" radius="0.05">
-            <origin xyz="0 0 0" rpy="0 0 0"/>
-        </xacro:inertial_sphere>
-    </link>
-    <gazebo reference="caster_wheel">
-        <material>Gazebo/Black</material>
-        <mu1 value="0.0000001" />
-        <mu2 value="0.0000001" />
-    </gazebo>
 </robot>
