Commit message: fix: correct URDF root link order, lidar sensor plugin, and scan bridge
Bug 1 — robot_core.xacro:
  base_footprint was declared after base_link. URDF parsers on ROS2 Foxy
  determine the root by finding a link with no parent joint. With base_link
  declared first some parsers treated it as root and published
  base_link→base_footprint (inverted), breaking the entire TF chain.
  Fix: declare base_footprint first, then base_link as its child.

Bug 2 — lidar.xacro:
  The sensor used type="ray" with libignition-gazebo-sensors-system.so as
  a per-sensor plugin. That plugin is a world-level system plugin, not a
  sensor plugin. It silently failed to publish /scan, so SLAM Toolbox
  received no laser data and never published the map→odom TF.
  Fix: change sensor type to gpu_lidar, use the correct
  libignition-gazebo-gpu-rays-system.so plugin, output on topic /scan
  with frame_id laser_frame.

Bug 3 — gz.launch.py:
  Scan bridge used ignition.msgs.LaserScan which only works with ray type.
  gpu_lidar publishes on ignition.msgs.LaserScan too but the topic name
  inside Ignition is /model/mobile_robot/laser — not /scan.
  Fix: bridge the model-namespaced Ignition topic to /scan on the ROS side
  using the correct remapping notation.

File: description/xacro/lidar.xacro (robot description, xacro)
@@ -1,7 +1,7 @@
 <?xml version="1.0"?>
-<robot xmlns:xacro="http://www.ros.org/wiki/xacro" >
+<robot xmlns:xacro="http://www.ros.org/wiki/xacro">
     <joint name="laser_joint" type="fixed">
         <parent link="chassis"/>
-        <child link="laser_frame"/>
+        <child  link="laser_frame"/>
         <origin xyz="0.122 0 0.212" rpy="0 0 0"/>
     </joint>
@@ -29,29 +29,51 @@
         </xacro:inertial_cylinder>
     </link>
+    <!--
+        Ignition Fortress lidar sensor.
+        Use sensor type="gpu_lidar" (not "ray").
+        "ray" is the Gazebo Classic type and does NOT work in Ignition.
+        The plugin that drives the sensor is libignition-gazebo-gpu-rays-system.so
+        loaded via the <sensor> block. The world must also load the
+        Sensors world-level system plugin (libignition-gazebo-sensors-system.so)
+        in the .world file — without it every sensor in the world is silent.
+        Topic remapping:
+          Ignition publishes on:  /world/<world>/model/mobile_robot/link/laser_frame/sensor/laser/scan
+          The gz.launch.py bridge maps this to ROS topic: /scan
+          SLAM Toolbox subscribes to: /scan
+    -->
     <gazebo reference="laser_frame">
         <material>Gazebo/Red</material>
-        <sensor name="laser" type="ray">
-            <pose> 0 0 0 0 0 0 </pose>
+        <sensor name="laser" type="gpu_lidar">
+            <pose>0 0 0 0 0 0</pose>
             <visualize>false</visualize>
             <update_rate>10</update_rate>
-            <ray>
+            <lidar>
                 <scan>
                     <horizontal>
                         <samples>360</samples>
-                        <min_angle>-3.14</min_angle>
-                        <max_angle>3.14</max_angle>
+                        <resolution>1</resolution>
+                        <min_angle>-3.14159</min_angle>
+                        <max_angle>3.14159</max_angle>
                     </horizontal>
                 </scan>
                 <range>
                     <min>0.3</min>
-                    <max>12</max>
+                    <max>12.0</max>
+                    <resolution>0.01</resolution>
                 </range>
-            </ray>
-            <plugin name="ignition::gazebo::systems::Sensors" filename="libignition-gazebo-sensors-system.so">
-                <ros>
-                    <argument> ~/out:=scan</argument>
-                </ros>
+            </lidar>
+            <!--
+                topic: the short name published inside Ignition.
+                The full Ignition topic will be:
+                  /world/<world_name>/model/mobile_robot/link/laser_frame/sensor/laser/scan
+                gz.launch.py bridges this to the ROS topic /scan.
+                frame_id must match the URDF link name so LaserScan
+                messages carry the correct TF frame.
+            -->
+            <plugin name="ignition::gazebo::systems::GpuLidar"
+                    filename="libignition-gazebo-gpu-rays-system.so">
+                <topic>scan</topic>
+                <frame_id>laser_frame</frame_id>
                 <output_type>sensor_msgs/LaserScan</output_type>
-                <frame_name>laser_frame</frame_name>
             </plugin>
         </sensor>

File: description/xacro/robot_core.xacro (robot description, xacro)
@@ -8,16 +8,27 @@
     <xacro:include filename="$(find mobile_robot)/description/xacro/left_wheels.xacro" />
     <xacro:include filename="$(find mobile_robot)/description/xacro/right_wheels.xacro" />
-    <!-- Base link -->
-    <link name="base_link"></link>
+    <!--
+        IMPORTANT: base_footprint MUST be declared first so that every URDF
+        parser (including ROS2 Foxy's urdf_parser) correctly identifies it as
+        the root link. The root is determined by finding a link that never
+        appears as a <child> in any joint. If base_link is declared first,
+        older parsers may pick it as root and publish base_link→base_footprint
+        (inverted), which breaks the entire TF chain:
+          map → odom → base_footprint → base_link  (correct)
+          map → odom → base_link → base_footprint  (WRONG — breaks Nav2 / SLAM)
+    -->
+    <!-- Virtual root link: no geometry, no inertia, sits on the ground plane -->
+    <link name="base_footprint"/>
+    <!-- base_footprint → base_link (fixed, zero offset) -->
     <joint name="base_footprint_joint" type="fixed">
-        <child link="base_link" />
         <parent link="base_footprint"/>
+        <child  link="base_link"/>
         <origin xyz="0 0 0" rpy="0 0 0"/>
     </joint>
-    <link name="base_footprint"></link>
-    <!-- Chassis -->
+    <link name="base_link"/>
+    <!-- base_link → chassis -->
     <joint name="chassis_joint" type="fixed">
-        <parent link="base_link" />
-        <child link="chassis" />
+        <parent link="base_link"/>
+        <child  link="chassis"/>
         <origin xyz="-0.1 0 0"/>
     </joint>
