Commit message: not turning issue fixed

File: description/xacro/left_wheels.xacro (robot description, xacro)
@@ -69,7 +69,7 @@
         <material>Gazebo/Black</material>
         <mu>1.0</mu>
-        <mu2>0.5</mu2>
-        <kp>1000000.0</kp>
-        <kd>1.0</kd>
+        <mu1>1.0</mu1>
+        <mu2>0.2</mu2>
+        <fdir1>1 0 0</fdir1>
         <minDepth>0.001</minDepth>
     </gazebo>
@@ -77,7 +77,7 @@
         <material>Gazebo/Black</material>
         <mu>1.0</mu>
-        <mu2>0.5</mu2>
-        <kp>1000000.0</kp>
-        <kd>1.0</kd>
+        <mu1>1.0</mu1>
+        <mu2>0.2</mu2>
+        <fdir1>1 0 0</fdir1>
         <minDepth>0.001</minDepth>
     </gazebo>

File: description/xacro/right_wheels.xacro (robot description, xacro)
@@ -25,16 +25,4 @@
         </xacro:inertial_cylinder>
     </link>
-    <!--
-         Ignition Gazebo friction and contact properties for right wheels.
-         See left_wheels.xacro for full parameter rationale.
-    -->
-    <gazebo reference="front_right_wheel">
-        <material>Gazebo/Black</material>
-        <mu>1.0</mu>
-        <mu2>0.5</mu2>
-        <kp>1000000.0</kp>
-        <kd>1.0</kd>
-        <minDepth>0.001</minDepth>
-    </gazebo>
     <!-- Rear wheel -->
     <joint name="rear_right_wheel_joint" type="continuous">
@@ -60,10 +48,22 @@
         </xacro:inertial_cylinder>
     </link>
+    <!--
+         Ignition Gazebo friction and contact properties for right wheels.
+         See left_wheels.xacro for full parameter rationale.
+    -->
+    <gazebo reference="front_right_wheel">
+        <material>Gazebo/Black</material>
+        <mu>1.0</mu>
+        <mu1>1.0</mu1>
+        <mu2>0.2</mu2>
+        <fdir1>1 0 0</fdir1>
+        <minDepth>0.001</minDepth>
+    </gazebo>
     <gazebo reference="rear_right_wheel">
         <material>Gazebo/Black</material>
         <mu>1.0</mu>
-        <mu2>0.5</mu2>
-        <kp>1000000.0</kp>
-        <kd>1.0</kd>
+        <mu1>1.0</mu1>
+        <mu2>0.2</mu2>
+        <fdir1>1 0 0</fdir1>
         <minDepth>0.001</minDepth>
     </gazebo>

File: description/xacro/ros2_control.xacro (robot description, xacro)
@@ -26,6 +26,6 @@
             <joint name="front_left_wheel_joint">
                 <command_interface name="velocity">
-                    <param name="min">-10</param>
-                    <param name="max">10</param>
+                    <param name="min">-20</param>
+                    <param name="max">20</param>
                 </command_interface>
                 <state_interface name="velocity"/>
@@ -34,6 +34,6 @@
             <joint name="front_right_wheel_joint">
                 <command_interface name="velocity">
-                    <param name="min">-10</param>
-                    <param name="max">10</param>
+                    <param name="min">-20</param>
+                    <param name="max">20</param>
                 </command_interface>
                 <state_interface name="velocity"/>
@@ -42,6 +42,6 @@
             <joint name="rear_left_wheel_joint">
                 <command_interface name="velocity">
-                    <param name="min">-10</param>
-                    <param name="max">10</param>
+                    <param name="min">-20</param>
+                    <param name="max">20</param>
                 </command_interface>
                 <state_interface name="velocity"/>
@@ -50,6 +50,6 @@
             <joint name="rear_right_wheel_joint">
                 <command_interface name="velocity">
-                    <param name="min">-10</param>
-                    <param name="max">10</param>
+                    <param name="min">-20</param>
+                    <param name="max">20</param>
                 </command_interface>
                 <state_interface name="velocity"/>
@@ -72,6 +72,6 @@
             <joint name="front_left_wheel_joint">
                 <command_interface name="velocity">
-                    <param name="min">-10</param>
-                    <param name="max">10</param>
+                    <param name="min">-20</param>
+                    <param name="max">20</param>
                 </command_interface>
                 <state_interface name="velocity"/>
@@ -80,6 +80,6 @@
             <joint name="front_right_wheel_joint">
                 <command_interface name="velocity">
-                    <param name="min">-10</param>
-                    <param name="max">10</param>
+                    <param name="min">-20</param>
+                    <param name="max">20</param>
                 </command_interface>
                 <state_interface name="velocity"/>
@@ -88,6 +88,6 @@
             <joint name="rear_left_wheel_joint">
                 <command_interface name="velocity">
-                    <param name="min">-10</param>
-                    <param name="max">10</param>
+                    <param name="min">-20</param>
+                    <param name="max">20</param>
                 </command_interface>
                 <state_interface name="velocity"/>
@@ -96,6 +96,6 @@
             <joint name="rear_right_wheel_joint">
                 <command_interface name="velocity">
-                    <param name="min">-10</param>
-                    <param name="max">10</param>
+                    <param name="min">-20</param>
+                    <param name="max">20</param>
                 </command_interface>
                 <state_interface name="velocity"/>

Commit message: change wheels to mecanum wheels

File: description/xacro/left_wheels.xacro (robot description, xacro)
@@ -1,6 +1,15 @@
 <?xml version="1.0"?>
-<robot xmlns:xacro="http://www.ros.org/wiki/xacro" >
+<robot xmlns:xacro="http://www.ros.org/wiki/xacro"
+       xmlns:ignition="http://gazebosim.org/schema">
+    <!--
+        xmlns:ignition namespace above is REQUIRED for the
+        <fdir1 ignition:expressed_in="..."> attribute below to survive
+        xacro processing. On Gazebo Fortress the attribute is
+        "ignition:expressed_in" (Garden+ renames it "gz:expressed_in").
+        NOTE: this declaration must ALSO exist on your main/top-level
+        robot xacro's <robot> tag - see right_wheels.xacro notes.
+    -->
     <xacro:include filename="$(find mobile_robot)/description/xacro/inertial_macros.xacro" />
-    <!-- Front wheel -->
+    <!-- Front left wheel -->
     <joint name="front_left_wheel_joint" type="continuous">
         <parent link="chassis" />
@@ -25,5 +34,5 @@
         </xacro:inertial_cylinder>
     </link>
-    <!-- Rear wheel -->
+    <!-- Rear left wheel -->
     <joint name="rear_left_wheel_joint" type="continuous">
         <parent link="chassis" />
@@ -48,9 +57,48 @@
         </xacro:inertial_cylinder>
     </link>
+    <!--
+        Mecanum roller friction emulation (Gazebo Fortress / ODE physics).
+        See right_wheels.xacro for full parameter rationale.
+        Roller pairing is DIAGONAL, matching the right side:
+          front_left  + rear_right -> Type A, fdir1 = "1  1 0"
+          rear_left   + front_right -> Type B, fdir1 = "1 -1 0"
+    -->
+    <gazebo reference="front_left_wheel">
+        <material>Gazebo/Black</material>
+        <collision>
+            <surface>
+                <friction>
+                    <ode>
+                        <mu>1.0</mu>
+                        <mu2>0.02</mu2>
+                        <fdir1 ignition:expressed_in="chassis">1 1 0</fdir1>
+                    </ode>
+                </friction>
+                <contact>
+                    <ode>
+                        <min_depth>0.001</min_depth>
+                    </ode>
+                </contact>
+            </surface>
+        </collision>
+    </gazebo>
     <gazebo reference="rear_left_wheel">
         <material>Gazebo/Black</material>
-    </gazebo>
-    <gazebo reference="front_left_wheel">
-        <material>Gazebo/Black</material>
+        <collision>
+            <surface>
+                <friction>
+                    <ode>
+                        <mu>1.0</mu>
+                        <mu2>0.02</mu2>
+                        <fdir1 ignition:expressed_in="chassis">1 -1 0</fdir1>
+                    </ode>
+                </friction>
+                <contact>
+                    <ode>
+                        <min_depth>0.001</min_depth>
+                    </ode>
+                </contact>
+            </surface>
+        </collision>
     </gazebo>
 </robot>

File: description/xacro/right_wheels.xacro (robot description, xacro)
@@ -1,6 +1,13 @@
 <?xml version="1.0"?>
-<robot xmlns:xacro="http://www.ros.org/wiki/xacro" >
+<robot xmlns:xacro="http://www.ros.org/wiki/xacro"
+       xmlns:ignition="http://gazebosim.org/schema">
+    <!--
+        xmlns:ignition namespace above is REQUIRED for the
+        <fdir1 ignition:expressed_in="..."> attribute below to survive
+        xacro processing. On Gazebo Fortress the attribute is
+        "ignition:expressed_in" (Garden+ renames it "gz:expressed_in").
+    -->
     <xacro:include filename="$(find mobile_robot)/description/xacro/inertial_macros.xacro" />
-    <!-- Front wheel -->
+    <!-- Front right wheel -->
     <joint name="front_right_wheel_joint" type="continuous">
         <parent link="chassis" />
@@ -25,8 +32,5 @@
         </xacro:inertial_cylinder>
     </link>
-    <gazebo reference="front_right_wheel">
-        <material>Gazebo/Black</material>
-    </gazebo>
-    <!-- Rear wheel -->
+    <!-- Rear right wheel -->
     <joint name="rear_right_wheel_joint" type="continuous">
         <parent link="chassis" />
@@ -51,6 +55,56 @@
         </xacro:inertial_cylinder>
     </link>
+    <!--
+        Mecanum roller friction emulation (Gazebo Fortress / ODE physics).
+        Real 45-deg rollers are NOT modeled as geometry here - instead we
+        keep the plain cylinder collision and fake roller behavior with
+        anisotropic friction:
+          - mu1 (high, along fdir1) = the wheel's effective push direction,
+            i.e. the direction force actually gets transmitted to the ground.
+          - mu2 (near zero, auto-computed orthogonal to fdir1) = the
+            roller's free-slip axis, letting the wheel "skate" sideways.
+        Roller pairing is DIAGONAL, not left/right:
+          front_right + rear_left   -> Type B, fdir1 = "1 -1 0"
+          front_left  + rear_right  -> Type A, fdir1 = "1  1 0"
+        fdir1 is expressed_in="chassis" so the vector means the same thing
+        regardless of each wheel link's own rotated joint frame.
+    -->
+    <gazebo reference="front_right_wheel">
+        <material>Gazebo/Black</material>
+        <collision>
+            <surface>
+                <friction>
+                    <ode>
+                        <mu>1.0</mu>
+                        <mu2>0.02</mu2>
+                        <fdir1 ignition:expressed_in="chassis">1 -1 0</fdir1>
+                    </ode>
+                </friction>
+                <contact>
+                    <ode>
+                        <min_depth>0.001</min_depth>
+                    </ode>
+                </contact>
+            </surface>
+        </collision>
+    </gazebo>
     <gazebo reference="rear_right_wheel">
         <material>Gazebo/Black</material>
+        <collision>
+            <surface>
+                <friction>
+                    <ode>
+                        <mu>1.0</mu>
+                        <mu2>0.02</mu2>
+                        <fdir1 ignition:expressed_in="chassis">1 1 0</fdir1>
+                    </ode>
+                </friction>
+                <contact>
+                    <ode>
+                        <min_depth>0.001</min_depth>
+                    </ode>
+                </contact>
+            </surface>
+        </collision>
     </gazebo>
 </robot>

Commit message: fix: normalize fdir1 vectors, add ignition namespace, validate duration, guard cmd-topic subscriber and shutdown race

File: description/xacro/left_wheels.xacro (robot description, xacro)
@@ -61,6 +61,9 @@
         See right_wheels.xacro for full parameter rationale.
         Roller pairing is DIAGONAL, matching the right side:
-          front_left  + rear_right -> Type A, fdir1 = "1  1 0"
-          rear_left   + front_right -> Type B, fdir1 = "1 -1 0"
+          front_left  + rear_right -> Type A, fdir1 = "0.70710678  0.70710678 0"
+          rear_left   + front_right -> Type B, fdir1 = "0.70710678 -0.70710678 0"
+        fdir1 is normalized to unit length (1/sqrt(2) ~= 0.70710678) since
+        Gazebo/ODE expects fdir1 to be a unit vector; an un-normalized
+        vector implicitly rescales the friction cone.
     -->
     <gazebo reference="front_left_wheel">
@@ -72,5 +75,5 @@
                         <mu>1.0</mu>
                         <mu2>0.02</mu2>
-                        <fdir1 ignition:expressed_in="chassis">1 1 0</fdir1>
+                        <fdir1 ignition:expressed_in="chassis">0.70710678 0.70710678 0</fdir1>
                     </ode>
                 </friction>
@@ -91,5 +94,5 @@
                         <mu>1.0</mu>
                         <mu2>0.02</mu2>
-                        <fdir1 ignition:expressed_in="chassis">1 -1 0</fdir1>
+                        <fdir1 ignition:expressed_in="chassis">0.70710678 -0.70710678 0</fdir1>
                     </ode>
                 </friction>

File: description/xacro/right_wheels.xacro (robot description, xacro)
@@ -65,8 +65,10 @@
             roller's free-slip axis, letting the wheel "skate" sideways.
         Roller pairing is DIAGONAL, not left/right:
-          front_right + rear_left   -> Type B, fdir1 = "1 -1 0"
-          front_left  + rear_right  -> Type A, fdir1 = "1  1 0"
+          front_right + rear_left   -> Type B, fdir1 = "0.70710678 -0.70710678 0"
+          front_left  + rear_right  -> Type A, fdir1 = "0.70710678  0.70710678 0"
         fdir1 is expressed_in="chassis" so the vector means the same thing
-        regardless of each wheel link's own rotated joint frame.
+        regardless of each wheel link's own rotated joint frame. It is
+        normalized to unit length (1/sqrt(2) ~= 0.70710678) since
+        Gazebo/ODE expects fdir1 to be a unit vector.
     -->
     <gazebo reference="front_right_wheel">
@@ -78,5 +80,5 @@
                         <mu>1.0</mu>
                         <mu2>0.02</mu2>
-                        <fdir1 ignition:expressed_in="chassis">1 -1 0</fdir1>
+                        <fdir1 ignition:expressed_in="chassis">0.70710678 -0.70710678 0</fdir1>
                     </ode>
                 </friction>
@@ -97,5 +99,5 @@
                         <mu>1.0</mu>
                         <mu2>0.02</mu2>
-                        <fdir1 ignition:expressed_in="chassis">1 1 0</fdir1>
+                        <fdir1 ignition:expressed_in="chassis">0.70710678 0.70710678 0</fdir1>
                     </ode>
                 </friction>

File: description/xacro/robot_core.xacro (robot description, xacro)
@@ -1,4 +1,5 @@
 <?xml version="1.0"?>
-<robot xmlns:xacro="http://www.ros.org/wiki/xacro">
+<robot xmlns:xacro="http://www.ros.org/wiki/xacro"
+       xmlns:ignition="http://gazebosim.org/schema">
     <xacro:include filename="$(find mobile_robot)/description/xacro/colors.xacro" />
     <xacro:include filename="$(find mobile_robot)/description/xacro/inertial_macros.xacro" />
@@ -8,6 +9,4 @@
     <xacro:include filename="$(find mobile_robot)/description/xacro/left_wheels.xacro" />
     <xacro:include filename="$(find mobile_robot)/description/xacro/right_wheels.xacro" />
-    <!-- IMU sensor: adds imu_link, imu_joint, and Ignition IMU plugin -->
-    <xacro:include filename="$(find mobile_robot)/description/xacro/imu.xacro" />
     <!--
         IMPORTANT: base_footprint MUST be declared first so that every URDF
@@ -37,14 +36,14 @@
     <link name="chassis">
         <visual>
-            <origin xyz="0.15 0 0.075" />
+            <origin xyz="0.15 0 0.075"/>
             <geometry>
-                <box size="0.3 0.3 0.15" />
+                <box size="0.3 0.3 0.15"/>
             </geometry>
-            <material name="white" />
+            <material name="white"/>
         </visual>
         <collision>
-            <origin xyz="0.15 0 0.075" />
+            <origin xyz="0.15 0 0.075"/>
             <geometry>
-                <box size="0.3 0.3 0.15" />
+                <box size="0.3 0.3 0.15"/>
             </geometry>
         </collision>
