Commit message: camera and lidar added

File: description/robot.urdf.xacro (robot description, xacro)
@@ -2,3 +2,4 @@
 <robot xmlns:xacro="http://www.ros.org/wiki/xacro"  name="robot">
      <xacro:include filename="$(find mobile_robot)/description/xacro/robot_core.xacro" />
+     <xacro:include filename="$(find mobile_robot)/description/xacro/gazebo_control.xacro"/>
 </robot>

File: description/xacro/robot_core.xacro (robot description, xacro)
@@ -1,6 +1,8 @@
 <?xml version="1.0"?>
-<robot xmlns:xacro="http://www.ros.org/wiki/xacro"  name="robot">
+<robot xmlns:xacro="http://www.ros.org/wiki/xacro">
     <xacro:include filename="$(find mobile_robot)/description/xacro/colors.xacro" />
     <xacro:include filename="$(find mobile_robot)/description/xacro/inertial_macros.xacro" />
+    <xacro:include filename="$(find mobile_robot)/description/xacro/lidar.xacro" />
+    <xacro:include filename="$(find mobile_robot)/description/xacro/camera.xacro" />
     <!-- Base link -->
     <link name="base_link"></link>
@@ -29,4 +31,7 @@
         </xacro:inertial_box>
     </link>
+    <gazebo reference="chassis">
+        <material>Gazebo/White</material>
+    </gazebo>
     <!-- Wheels -->
     <!-- Left wheel -->
@@ -53,4 +58,7 @@
         </xacro:inertial_cylinder>
     </link>
+    <gazebo reference="left_wheel">
+        <material>Gazebo/Black</material>
+    </gazebo>
     <!-- Right wheel -->
     <joint name="right_wheel_joint" type="continuous">
@@ -76,4 +84,7 @@
         </xacro:inertial_cylinder>
     </link>
+    <gazebo reference="right_wheel">
+        <material>Gazebo/Black</material>
+    </gazebo>
     <!-- Caster wheel -->
     <joint name="caster_wheel_joint" type="fixed">
@@ -98,3 +109,8 @@
         </xacro:inertial_sphere>
     </link>
+    <gazebo reference="caster_wheel">
+        <material>Gazebo/Black</material>
+        <mu1 value="0.0000001" />
+        <mu2 value="0.0000001" />
+    </gazebo>
 </robot>

Commit message: add joystick control

File: description/robot.urdf.xacro (robot description, xacro)
@@ -1,5 +1,13 @@
 <?xml version="1.0"?>
 <robot xmlns:xacro="http://www.ros.org/wiki/xacro"  name="robot">
+     <xacro:arg name="use_ros2_control" default="true"/>
+     <xacro:arg name="sim_mode" default="true"/>
      <xacro:include filename="$(find mobile_robot)/description/xacro/robot_core.xacro" />
-     <xacro:include filename="$(find mobile_robot)/description/xacro/gazebo_control.xacro"/>
+     <!-- <xacro:include filename="$(find mobile_robot)/description/xacro/gazebo_control.xacro"/> -->
+     <xacro:if value="$(arg use_ros2_control)">
+        <xacro:include filename="$(find mobile_robot)/description/xacro/ros2_control.xacro" />
+    </xacro:if>
+    <xacro:unless value="$(arg use_ros2_control)">
+        <xacro:include filename="$(find mobile_robot)/description/xacro/gazebo_control.xacro" />
+    </xacro:unless>
 </robot>

File: description/xacro/gazebo_control.xacro (robot description, xacro)
@@ -2,14 +2,32 @@
 <robot xmlns:xacro="http://www.ros.org/wiki/xacro">
     <gazebo>
-        <plugin name="motor_control" filename="libgazebo_ros_diff_drive.so">
+        <plugin name="front_motor_control" filename="libgazebo_ros_diff_drive.so">
             <!-- Front Wheels -->
             <left_joint>front_left_wheel_joint</left_joint>
             <right_joint>front_right_wheel_joint</right_joint>
-            <!-- Rear Wheels -->
-            <left_rear_joint>rear_left_wheel_joint</left_rear_joint>
-            <right_rear_joint>rear_right_wheel_joint</right_rear_joint>
             <!-- Wheel Configuration -->
             <wheel_separation>0.35</wheel_separation>
-            <wheel_diameter>0.1</wheel_diameter>
+            <wheel_diameter>0.048</wheel_diameter>
+            <!-- Limits -->
+            <max_wheel_torque>200</max_wheel_torque>
+            <wheel_acceleration>10.0</wheel_acceleration>
+            <!-- Output -->
+            <odometry_frame>odom</odometry_frame>
+            <robot_base_frame>base_link</robot_base_frame>
+            <!-- Publishing Options -->
+            <publish_odom>true</publish_odom>
+            <publish_odom_tf>true</publish_odom_tf>
+            <publish_wheel_tf>true</publish_wheel_tf>
+            <!-- Additional Parameters for 4 Wheels -->
+            <legacyMode>false</legacyMode>
+            <updateRate>50.0</updateRate>
+        </plugin>
+        <plugin name="rear_motor_control" filename="libgazebo_ros_diff_drive.so">
+            <!-- Rear Wheels -->
+            <left_joint>rear_left_wheel_joint</left_joint>
+            <right_joint>rear_right_wheel_joint</right_joint>
+            <!-- Wheel Configuration -->
+            <wheel_separation>0.35</wheel_separation>
+            <wheel_diameter>0.048</wheel_diameter>
             <!-- Limits -->
             <max_wheel_torque>200</max_wheel_torque>

File: description/xacro/left_wheels.xacro (robot description, xacro)
@@ -2,11 +2,4 @@
 <robot xmlns:xacro="http://www.ros.org/wiki/xacro" >
     <xacro:include filename="$(find mobile_robot)/description/xacro/inertial_macros.xacro" />
-    <!-- <joint name="front_left_joint" type="fixed">
-        <parent link="chassis" />
-        <child link="front_left" />
-        <origin xyz="0.25 0.175 0" rpy="-${pi/2} 0 0"/>
-        <axis xyz="0 0 1" />
-    </joint>
-    <link name="front_left"></link> -->
     <!-- Front wheel -->
     <joint name="front_left_wheel_joint" type="continuous">
@@ -19,5 +12,5 @@
         <visual>
             <geometry>
-                <cylinder radius="0.05" length="0.04" />
+                <cylinder radius="0.024" length="0.025" />
             </geometry>
             <material name="black" />
@@ -25,18 +18,11 @@
         <collision>
             <geometry>
-                <cylinder radius="0.05" length="0.04" />
+                <cylinder radius="0.024" length="0.025" />
             </geometry>
         </collision>
-        <xacro:inertial_cylinder mass="0.1" length="0.04" radius="0.05">
+        <xacro:inertial_cylinder mass="0.1" length="0.025" radius="0.024">
             <origin xyz="0 0 0" rpy="0 0 0"/>
         </xacro:inertial_cylinder>
     </link>
-    <!-- <joint name="rear_left_joint" type="fixed">
-        <parent link="chassis" />
-        <child link="rear_left" />
-        <origin xyz="0.05 0.175 0" rpy="-${pi/2} 0 0"/>
-        <axis xyz="0 0 1" />
-    </joint>
-    <link name="rear_left"></link> -->
     <!-- Rear wheel -->
     <joint name="rear_left_wheel_joint" type="continuous">
@@ -49,5 +35,5 @@
         <visual>
             <geometry>
-                <cylinder radius="0.05" length="0.04" />
+                <cylinder radius="0.024" length="0.025" />
             </geometry>
             <material name="black" />
@@ -55,8 +41,8 @@
         <collision>
             <geometry>
-                <cylinder radius="0.05" length="0.04" />
+                <cylinder radius="0.024" length="0.025" />
             </geometry>
         </collision>
-        <xacro:inertial_cylinder mass="0.1" length="0.04" radius="0.05">
+        <xacro:inertial_cylinder mass="0.1" length="0.025" radius="0.024">
             <origin xyz="0 0 0" rpy="0 0 0"/>
         </xacro:inertial_cylinder>

File: description/xacro/lidar.xacro (robot description, xacro)
@@ -50,5 +50,5 @@
             <plugin name="laser_controller" filename="libgazebo_ros_ray_sensor.so">
                 <ros>
-                    <argument>--ros-args --remap ~/out:=scan</argument>
+                    <argument>~/out:=scan</argument>
                 </ros>
                 <output_type>sensor_msgs/LaserScan</output_type>

File: description/xacro/right_wheels.xacro (robot description, xacro)
@@ -12,5 +12,5 @@
         <visual>
             <geometry>
-                <cylinder radius="0.05" length="0.04" />
+                <cylinder radius="0.024" length="0.025" />
             </geometry>
             <material name="black" />
@@ -18,8 +18,8 @@
         <collision>
             <geometry>
-                <cylinder radius="0.05" length="0.04" />
+                <cylinder radius="0.024" length="0.025" />
             </geometry>
         </collision>
-        <xacro:inertial_cylinder mass="0.1" length="0.04" radius="0.05">
+        <xacro:inertial_cylinder mass="0.1" length="0.025" radius="0.024">
             <origin xyz="0 0 0" rpy="0 0 0"/>
         </xacro:inertial_cylinder>
@@ -38,5 +38,5 @@
         <visual>
             <geometry>
-                <cylinder radius="0.05" length="0.04" />
+                <cylinder radius="0.024" length="0.025" />
             </geometry>
             <material name="black" />
@@ -44,8 +44,8 @@
         <collision>
             <geometry>
-                <cylinder radius="0.05" length="0.04" />
+                <cylinder radius="0.024" length="0.025" />
             </geometry>
         </collision>
-        <xacro:inertial_cylinder mass="0.1" length="0.04" radius="0.05">
+        <xacro:inertial_cylinder mass="0.1" length="0.025" radius="0.024">
             <origin xyz="0 0 0" rpy="0 0 0"/>
         </xacro:inertial_cylinder>

File: description/xacro/robot_core.xacro (robot description, xacro)
@@ -10,4 +10,10 @@
     <!-- Base link -->
     <link name="base_link"></link>
+    <joint name="base_footprint_joint" type="fixed">
+        <parent link="base_link" />
+        <child link="base_footprint"/>
+        <origin xyz="0 0 0" rpy="0 0 0"/>
+    </joint>
+    <link name="base_footprint"></link>
     <!-- Chassis -->
     <joint name="chassis_joint" type="fixed">

Commit message: add slam online async

File: description/robot.urdf.xacro (robot description, xacro)
@@ -1,13 +1,13 @@
 <?xml version="1.0"?>
-<robot xmlns:xacro="http://www.ros.org/wiki/xacro"  name="robot">
-     <xacro:arg name="use_ros2_control" default="true"/>
-     <xacro:arg name="sim_mode" default="true"/>
-     <xacro:include filename="$(find mobile_robot)/description/xacro/robot_core.xacro" />
-     <!-- <xacro:include filename="$(find mobile_robot)/description/xacro/gazebo_control.xacro"/> -->
-     <xacro:if value="$(arg use_ros2_control)">
+<robot xmlns:xacro="http://www.ros.org/wiki/xacro"  name="Mobile Robot">
+    <xacro:arg name="use_ros2_control" default="false"/>
+    <xacro:arg name="sim_mode" default="true"/>
+    <xacro:include filename="$(find mobile_robot)/description/xacro/robot_core.xacro" />
+    <!-- Control inclusion based on use_ros2_control argument -->
+    <xacro:if value="${'$(arg use_ros2_control)' == 'true'}">
         <xacro:include filename="$(find mobile_robot)/description/xacro/ros2_control.xacro" />
     </xacro:if>
-    <xacro:unless value="$(arg use_ros2_control)">
+    <xacro:if value="${'$(arg use_ros2_control)' == 'false'}">
         <xacro:include filename="$(find mobile_robot)/description/xacro/gazebo_control.xacro" />
-    </xacro:unless>
+    </xacro:if>
 </robot>

File: description/xacro/colors.xacro (robot description, xacro)
@@ -1,4 +1,4 @@
 <?xml version="1.0"?>
-<robot xmlns:xacro="http://www.ros.org/wiki/xacro"  name="robot">
+<robot xmlns:xacro="http://www.ros.org/wiki/xacro"  name="Mobile Robot">
     <material name="white">
         <color rgba="1 1 1 1"/>

File: description/xacro/lidar.xacro (robot description, xacro)
@@ -50,5 +50,5 @@
             <plugin name="laser_controller" filename="libgazebo_ros_ray_sensor.so">
                 <ros>
-                    <argument>~/out:=scan</argument>
+                    <argument> ~/out:=scan</argument>
                 </ros>
                 <output_type>sensor_msgs/LaserScan</output_type>

File: description/xacro/ros2_control.xacro (robot description, xacro)
@@ -5,6 +5,8 @@
             <hardware>
                 <plugin>diffdrive_arduino/DiffDriveArduino</plugin>
-                <param name="left_wheel_name">left_wheel_joint</param>
-                <param name="right_wheel_name">right_wheel_joint</param>
+                <param name="left_wheel_name">front_left_wheel_joint</param>
+                <param name="right_wheel_name">front_right_wheel_joint</param>
+                <param name="left_wheel_name">rear_left_wheel_joint</param>
+                <param name="right_wheel_name">rear_right_wheel_joint</param>
                 <param name="loop_rate">30</param>
                 <param name="device">/dev/ttyUSB0</param>
@@ -13,5 +15,5 @@
                 <param name="enc_counts_per_rev">3436</param>
             </hardware>
-            <joint name="left_wheel_joint">
+            <joint name="front_left_wheel_joint">
                 <command_interface name="velocity">
                     <param name="min">-10</param>
@@ -21,5 +23,21 @@
                 <state_interface name="position"/>
             </joint>
-            <joint name="right_wheel_joint">
+            <joint name="front_right_wheel_joint">
+                <command_interface name="velocity">
+                    <param name="min">-10</param>
+                    <param name="max">10</param>
+                </command_interface>
+                <state_interface name="velocity"/>
+                <state_interface name="position"/>
+            </joint>
+            <joint name="rear_left_wheel_joint">
+                <command_interface name="velocity">
+                    <param name="min">-10</param>
+                    <param name="max">10</param>
+                </command_interface>
+                <state_interface name="velocity"/>
+                <state_interface name="position"/>
+            </joint>
+            <joint name="rear_right_wheel_joint">
                 <command_interface name="velocity">
                     <param name="min">-10</param>
@@ -74,4 +92,7 @@
             <parameters>$(find mobile_robot)/config/controllers.yaml</parameters>
             <parameters>$(find mobile_robot)/config/gaz_ros2_ctl_use_sim.yaml</parameters>
+            <!-- <ros>
+                <namespace>mobile_robot</namespace>
+            </ros> -->
         </plugin>
     </gazebo>

Commit message: updated robot to use 3D lidar

File: description/robot.urdf.xacro (robot description, xacro)
@@ -3,4 +3,6 @@
     <xacro:arg name="use_ros2_control" default="false"/>
     <xacro:arg name="sim_mode" default="true"/>
+    <xacro:arg name="show_ray" default="false"/>
+    <xacro:arg name="show_camera" default="false"/>
     <xacro:include filename="$(find mobile_robot)/description/xacro/robot_core.xacro" />
     <!-- Control inclusion based on use_ros2_control argument -->

File: description/xacro/left_camera.xacro (robot description, xacro)
@@ -1,4 +1,5 @@
 <?xml version="1.0"?>
 <robot xmlns:xacro="http://www.ros.org/wiki/xacro" >
+    <xacro:property name="visualize" value="$(arg show_camera)"/>
     <joint name="left_camera_joint" type="fixed">
         <parent link="chassis"/>
@@ -31,5 +32,5 @@
         <sensor name="left_camera" type="camera">
             <pose> 0 0 0 0 0 0 </pose>
-            <visualize>true</visualize>
+            <visualize>${visualize}</visualize>
             <update_rate>10</update_rate>
             <camera>
@@ -46,5 +47,4 @@
             </camera>
             <plugin name="left_camera_controller" filename="libgazebo_ros_camera.so">
-                <!-- <robotNamespace>left_camera</robotNamespace> -->
                 <frame_name>left_camera_link_optical</frame_name>
             </plugin>

File: description/xacro/lidar.xacro (robot description, xacro)
@@ -1,4 +1,6 @@
 <?xml version="1.0"?>
 <robot xmlns:xacro="http://www.ros.org/wiki/xacro" >
+    <xacro:property name="visualize" value="$(arg show_ray)"/>
+    <xacro:property name="gpu" value="$(arg gpu_ray)"/>
     <joint name="laser_joint" type="fixed">
         <parent link="chassis"/>
@@ -31,29 +33,92 @@
     <gazebo reference="laser_frame">
         <material>Gazebo/Red</material>
-        <sensor name="laser" type="ray">
-            <pose> 0 0 0 0 0 0 </pose>
-            <visualize>false</visualize>
-            <update_rate>10</update_rate>
-            <ray>
-                <scan>
-                    <horizontal>
-                        <samples>360</samples>
-                        <min_angle>-3.14</min_angle>
-                        <max_angle>3.14</max_angle>
-                    </horizontal>
-                </scan>
-                <range>
-                    <min>0.3</min>
-                    <max>12</max>
-                </range>
-            </ray>
-            <plugin name="laser_controller" filename="libgazebo_ros_ray_sensor.so">
-                <ros>
-                    <argument> ~/out:=scan</argument>
-                </ros>
-                <output_type>sensor_msgs/LaserScan</output_type>
-                <frame_name>laser_frame</frame_name>
-            </plugin>
-        </sensor>
+        <xacro:if value="${gpu}">
+            <sensor name="laser" type="gpu_ray">
+                <pose> 0 0 0 0 0 0 </pose>
+                <visualize>${visualize}</visualize>
+                <update_rate>10</update_rate>
+                <ray>
+                    <scan>
+                        <horizontal>
+                            <samples>720</samples>
+                            <resolution>1.0</resolution>
+                            <min_angle>-3.14</min_angle>
+                            <max_angle>3.14</max_angle>
+                        </horizontal>
+                        <vertical>
+                            <samples>64</samples>
+                            <resolution>1.0</resolution>
+                            <min_angle>-0.535</min_angle>
+                            <max_angle>0.186</max_angle>
+                        </vertical>
+                    </scan>
+                    <range>
+                        <min>0.3</min>
+                        <max>10.0</max>
+                        <resolution>0.01</resolution>
+                    </range>
+                    <noise>
+                        <type>gaussian</type>
+                        <mean>0.0</mean>
+                        <stddev>0.0</stddev>
+                    </noise>
+                </ray>
+                <plugin name="gazebo_ros_laser_controller" filename="libgazebo_ros_velodyne_gpu_laser.so">
+                    <ros>
+                        <argument> ~/out:=scan</argument>
+                    </ros>
+                    <output_type>sensor_msgs/PointCloud2</output_type>
+                    <frame_name>laser_frame</frame_name>
+                    <organize_cloud>true</organize_cloud>
+                    <min_range>0.9</min_range>
+                    <max_range>12.0</max_range>
+                    <gaussian_noise>0.008</gaussian_noise>
+                </plugin>
+            </sensor>
+        </xacro:if>
+        <xacro:unless value="${gpu}">
+            <sensor name="laser" type="ray">
+                <pose> 0 0 0 0 0 0 </pose>
+                <visualize>${visualize}</visualize>
+                <update_rate>10</update_rate>
+                <ray>
+                    <scan>
+                        <horizontal>
+                            <samples>720</samples>
+                            <resolution>1.0</resolution>
+                            <min_angle>-3.14</min_angle>
+                            <max_angle>3.14</max_angle>
+                        </horizontal>
+                        <vertical>
+                            <samples>64</samples>
+                            <resolution>1.0</resolution>
+                            <min_angle>-0.535</min_angle>
+                            <max_angle>0.186</max_angle>
+                        </vertical>
+                    </scan>
+                    <range>
+                        <min>0.3</min>
+                        <max>10.0</max>
+                        <resolution>0.01</resolution>
+                    </range>
+                    <noise>
+                        <type>gaussian</type>
+                        <mean>0.0</mean>
+                        <stddev>0.0</stddev>
+                    </noise>
+                </ray>
+                <plugin name="gazebo_ros_laser_controller" filename="libgazebo_ros_velodyne_laser.so">
+                    <ros>
+                        <argument> ~/out:=scan</argument>
+                    </ros>
+                    <output_type>sensor_msgs/PointCloud2</output_type>
+                    <frame_name>laser_frame</frame_name>
+                    <organize_cloud>true</organize_cloud>
+                    <min_range>0.9</min_range>
+                    <max_range>12.0</max_range>
+                    <gaussian_noise>0.008</gaussian_noise>
+                </plugin>
+            </sensor>
+        </xacro:unless>
     </gazebo>
 </robot>

File: description/xacro/right_camera.xacro (robot description, xacro)
@@ -1,4 +1,5 @@
 <?xml version="1.0"?>
 <robot xmlns:xacro="http://www.ros.org/wiki/xacro" >
+    <xacro:property name="visualize" value="$(arg show_camera)"/>
     <joint name="right_camera_joint" type="fixed">
         <parent link="chassis"/>
@@ -31,5 +32,5 @@
         <sensor name="right_camera" type="camera">
             <pose> 0 0 0 0 0 0 </pose>
-            <visualize>true</visualize>
+            <visualize>${visualize}</visualize>
             <update_rate>10</update_rate>
             <camera>
@@ -46,5 +47,4 @@
             </camera>
             <plugin name="right_camera_controller" filename="libgazebo_ros_camera.so">
-                <!-- <robotNamespace>right_camera</robotNamespace> -->
                 <frame_name>right_camera_link_optical</frame_name>
             </plugin>

File: description/xacro/robot_core.xacro (robot description, xacro)
@@ -4,6 +4,6 @@
     <xacro:include filename="$(find mobile_robot)/description/xacro/inertial_macros.xacro" />
     <xacro:include filename="$(find mobile_robot)/description/xacro/lidar.xacro" />
-    <xacro:include filename="$(find mobile_robot)/description/xacro/right_camera.xacro" />
-    <xacro:include filename="$(find mobile_robot)/description/xacro/left_camera.xacro" />
+    <!-- <xacro:include filename="$(find mobile_robot)/description/xacro/right_camera.xacro"/>  -->
+    <!-- <xacro:include filename="$(find mobile_robot)/description/xacro/left_camera.xacro"/>  -->
     <xacro:include filename="$(find mobile_robot)/description/xacro/left_wheels.xacro" />
     <xacro:include filename="$(find mobile_robot)/description/xacro/right_wheels.xacro" />
