Commit message: fixing bugs

File: description/robot.urdf.xacro (robot description, xacro)
@@ -5,9 +5,9 @@
     <xacro:include filename="$(find mobile_robot)/description/xacro/robot_core.xacro" />
     <!-- Control inclusion based on use_ros2_control argument -->
-    <xacro:if value="${'$(arg use_ros2_control)' == 'true'}">
+    <xacro:if value="$(arg use_ros2_control)">
         <xacro:include filename="$(find mobile_robot)/description/xacro/ros2_control.xacro" />
     </xacro:if>
-    <xacro:if value="${'$(arg use_ros2_control)' == 'false'}">
+    <xacro:unless value="$(arg use_ros2_control)">
         <xacro:include filename="$(find mobile_robot)/description/xacro/gazebo_control.xacro" />
-    </xacro:if>
+    </xacro:unless>
 </robot>

File: description/xacro/robot_core.xacro (robot description, xacro)
@@ -11,6 +11,6 @@
     <link name="base_link"></link>
     <joint name="base_footprint_joint" type="fixed">
-        <parent link="base_link" />
-        <child link="base_footprint"/>
+        <child link="base_link" />
+        <parent link="base_footprint"/>
         <origin xyz="0 0 0" rpy="0 0 0"/>
     </joint>
